File: PCB/litl.kicad_sch (KiCad schematic)
At the start: 103 parts, among them J1 Conn_01x04, SW1 KEYSW, SW10 KEYSW, SW11 KEYSW, SW12 KEYSW, SW13 KEYSW, SW14 KEYSW, SW15 KEYSW, SW16 KEYSW, SW17 KEYSW, SW18 KEYSW, SW19 KEYSW, SW2 KEYSW, SW20 KEYSW, SW21 KEYSW, SW22 KEYSW, SW23 KEYSW, SW24 KEYSW, SW25 KEYSW, SW26 KEYSW, SW27 KEYSW, SW28 KEYSW, SW29 KEYSW, SW3 KEYSW, SW30 KEYSW, SW31 KEYSW, SW32 KEYSW, SW33 KEYSW, SW34 KEYSW, SW35 KEYSW, SW36 KEYSW, SW37 KEYSW, SW38 KEYSW, SW39 KEYSW, SW4 KEYSW, SW40 KEYSW, SW41 KEYSW, SW42 KEYSW, SW43 KEYSW, SW44 KEYSW, SW45 KEYSW, SW46 KEYSW, SW47 KEYSW, SW48 KEYSW, SW49 KEYSW, SW5 KEYSW, SW50 KEYSW, SW51 RotaryEncoder_Switch, SW52 KEYSW, SW53 RotaryEncoder_Switch, SW54 KEYSW, SW6 KEYSW, SW7 KEYSW, SW8 KEYSW, SW9 KEYSW, U1 ProMicro

Commit message: Ortho low profile gateron
Parts:
- removed SW15: KEYSW, Button_Switch_Keyboard:SW_Cherry_MX_1.00u_PCB, symbol keyboard_parts:KEYSW
- removed SW26: KEYSW, Button_Switch_Keyboard:SW_Cherry_MX_2.25u_PCB, symbol keyboard_parts:KEYSW
- removed SW28, SW45: KEYSW, Button_Switch_Keyboard:SW_Cherry_MX_1.25u_PCB, symbol keyboard_parts:KEYSW
- removed SW47: KEYSW, Button_Switch_Keyboard:SW_Cherry_MX_6.25u_PCB, symbol keyboard_parts:KEYSW
- added D48: D_Small, Keebio-Parts:Diode, symbol Device:D_Small
- added SW55: KEYSW, key-switches:SW_Gateron_LowProfile_THT180, symbol keyboard_parts:KEYSW
- SW1: footprint Button_Switch_Keyboard:SW_Cherry_MX_1.50u_Plate -> key-switches:SW_Gateron_LowProfile_THT180
- SW10, SW11, SW16, SW17, SW18, SW19, SW2, SW20, SW21, SW22, SW23, SW24, SW25, SW29, SW3, SW30, SW31, SW32, SW33, SW34, SW35, SW36, SW37, SW38, SW4, SW40, SW41, SW44, SW49, SW5, SW6, SW7, SW8, SW9: footprint Button_Switch_Keyboard:SW_Cherry_MX_1.00u_PCB -> key-switches:SW_Gateron_LowProfile_THT180
- SW12: footprint Button_Switch_Keyboard:SW_Cherry_MX_1.50u_PCB -> key-switches:SW_Gateron_LowProfile_THT180
- SW13, SW42, SW43, SW50, SW52: footprint Button_Switch_Keyboard:SW_Cherry_MX_1.25u_PCB -> key-switches:SW_Gateron_LowProfile_THT180
- SW14, SW39: footprint Button_Switch_Keyboard:SW_Cherry_MX_1.75u_PCB -> key-switches:SW_Gateron_LowProfile_THT180
- SW27, SW46: footprint Button_Switch_Keyboard:SW_Cherry_MX_2.25u_PCB -> key-switches:SW_Gateron_LowProfile_THT180
- SW48: footprint Button_Switch_Keyboard:SW_Cherry_MX_2.75u_PCB -> key-switches:SW_Gateron_LowProfile_THT180
Connections:
- net rowB is gone; now on net rowA: D10.1 (K), D12.1 (K), D2.1 (K), D4.1 (K), D6.1 (K), D8.1 (K), U1.12 (9/PB5)
- net rowD is gone; now on net rowC: D15.1 (K), D17.1 (K), D19.1 (K), D21.1 (K), D23.1 (K), D24.1 (K), U1.8 (5/PC6)
- net rowF is gone; now on net rowE: D26.1 (K), D28.1 (K), D30.1 (K), D32.1 (K), D34.1 (K), D36.1 (K), U1.10 (7/PE6)
- net rowH is gone; now on net rowG: D37.1 (K), D39.1 (K), D42.1 (K), D45.1 (K), D46.1 (K), U1.20 (A3/PF4)
- net col1: now also SW55.1
- net rowG: now also D48.1 (K)
- new net: D48.2 (A), SW55.2
Other:
- moved on the sheet: D1, D10, D11, D12, D13, D14, D17, D2, D21, D22, D24, D25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
