File: PCB/litl.kicad_pcb (KiCad board)
At the start: 2 copper layers, 248.3 x 99.8 mm, 168 parts, among them J1 Conn_01x04, SW1 KEYSW, SW10 GateronLP, SW10 KEYSW, SW11 GateronLP, SW11 KEYSW, SW12 GateronLP, SW12 KEYSW, SW13 KEYSW, SW14 GateronLP, SW14 KEYSW, SW15 GateronLP, SW16 GateronLP, SW16 KEYSW, SW17 GateronLP, SW17 KEYSW, SW18 GateronLP, SW18 KEYSW, SW19 KEYSW, SW2 GateronLP, SW2 KEYSW, SW20 GateronLP, SW20 KEYSW, SW21 GateronLP, SW21 KEYSW, SW22 GateronLP, SW22 KEYSW, SW23 GateronLP, SW23 KEYSW, SW24 GateronLP, SW24 KEYSW, SW25 KEYSW, SW27 KEYSW, SW29 KEYSW, SW3 GateronLP, SW3 KEYSW, SW30 KEYSW, SW31 KEYSW, SW32 KEYSW, SW33 KEYSW, SW34 KEYSW, SW35 KEYSW, SW36 KEYSW, SW37 KEYSW, SW38 KEYSW, SW39 KEYSW, SW4 GateronLP, SW4 KEYSW, SW40 KEYSW, SW41 KEYSW, SW42 KEYSW, SW43 KEYSW, SW44 KEYSW, SW46 KEYSW, SW48 KEYSW, SW49 KEYSW, SW5 GateronLP, SW5 KEYSW, SW50 KEYSW, SW51 RotaryEncoder_Switch, SW52 KEYSW, SW53 RotaryEncoder_Switch, SW54 KEYSW, SW55 KEYSW, SW6 GateronLP, SW6 KEYSW, SW7 KEYSW, SW8 GateronLP, SW8 KEYSW, SW9 GateronLP, SW9 KEYSW, U1 ProMicro

Commit message: production tweak
Routing:
- net RotC: track 83.3 -> 80.3 mm
- net Net-(D31-A): track 56.8 -> 56.2 mm
Changed lines of the file:
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@@
 	)
 	(segment
-		(start 56.945 28.4211)
-		(end 57.868111 27.497989)
-		(width 0.254)
-		(layer "B.Cu")
-		(net 1)
-	)
-	(segment
 		(start 86.915 28.65)
 		(end 88.067011 29.802011)
@@
 	)
 	(segment
-		(start 56.065011 29.623911)
-		(end 62.066089 29.623911)
-		(width 0.254)
-		(layer "B.Cu")
-		(net 1)
-	)
-	(segment
 		(start 147.754511 27.497989)
 		(end 169.325489 27.497989)
@@
 	)
 	(segment
-		(start 73.825489 27.497989)
-		(end 74.9775 28.65)
-		(width 0.254)
-		(layer "B.Cu")
-		(net 1)
-	)
-	(segment
 		(start 146.6025 28.65)
 		(end 147.754511 27.497989)
@@
 	)
 	(segment
-		(start 54.405 27.9639)
-		(end 56.065011 29.623911)
+		(start 170.4775 28.65)
+		(end 171.629511 27.497989)
 		(width 0.254)
 		(layer "B.Cu")
@@
 	)
 	(segment
-		(start 170.4775 28.65)
-		(end 171.629511 27.497989)
+		(start 54.405 27.9639)
+		(end 56.065011 29.623911)
 		(width 0.254)
 		(layer "B.Cu")
@@
 	)
 	(segment
-		(start 85.762989 29.802011)
-		(end 86.915 28.65)
+		(start 62.066089 29.623911)
+		(end 63.04 28.65)
 		(width 0.254)
 		(layer "B.Cu")
@@
 	)
 	(segment
-		(start 157.387989 29.802011)
-		(end 158.54 28.65)
+		(start 56.945 28.4211)
+		(end 57.868111 27.497989)
 		(width 0.254)
 		(layer "B.Cu")
@@
 	)
 	(segment
-		(start 57.868111 27.497989)
-		(end 73.825489 27.497989)
+		(start 85.762989 29.802011)
+		(end 86.915 28.65)
+		(width 0.254)
+		(layer "B.Cu")
+		(net 1)
+	)
+	(segment
+		(start 157.387989 29.802011)
+		(end 158.54 28.65)
 		(width 0.254)
 		(layer "B.Cu")
@@
 	)
 	(segment
-		(start 62.066089 29.623911)
-		(end 63.04 28.65)
+		(start 57.868111 27.497989)
+		(end 73.825489 27.497989)
+		(width 0.254)
+		(layer "B.Cu")
+		(net 1)
+	)
+	(segment
+		(start 56.065011 29.623911)
+		(end 62.066089 29.623911)
 		(width 0.254)
 		(layer "B.Cu")
@@
 	)
 	(segment
+		(start 73.825489 27.497989)
+		(end 74.9775 28.65)
+		(width 0.254)
+		(layer "B.Cu")
+		(net 1)
+	)
+	(segment
 		(start 159.692011 29.802011)
 		(end 181.262989 29.802011)
@@
 	)
 	(segment
-		(start 40.74 68.78)
-		(end 40.74 68.9325)
-		(width 0.25)
-		(locked yes)
-		(layer "F.Cu")
-		(net 13)
-	)
-	(segment
 		(start 65.9 72.3)
 		(end 65.9 91.3)
@@
 	)
 	(segment
-		(start 142 110.2)
-		(end 141.9 110.3)
-		(width 0.25)
-		(layer "B.Cu")
-		(net 15)
-	)
-	(segment
 		(start 141.9 72.3)
 		(end 141.9 84.76)
@@
 	)
 	(segment
-		(start 235.7 111.5)
-		(end 236.9 110.3)
-		(width 0.25)
-		(layer "B.Cu")
-		(net 17)
-	)
-	(segment
 		(start 59.40094 48.65704)
 		(end 54.405 43.6611)
@@
 	)
 	(segment
-		(start 226.48 111.5)
-		(end 235.7 111.5)
-		(width 0.25)
-		(layer "B.Cu")
-		(net 17)
-	)
-	(segment
 		(start 222.72 110.3)
 		(end 223.5 109.52)
@@
 	)
 	(segment
-		(start 224.12 109.52)
-		(end 224.5 109.52)
-		(width 0.25)
-		(locked yes)
-		(layer "B.Cu")
-		(net 17)
-	)
-	(segment
 		(start 198.9 52.805)
 		(end 194.75204 48.65704)
@@
 	)
 	(segment
-		(start 217.9 110.3)
-		(end 217.9 91.3)
+		(start 224.5 109.52)
+		(end 226.48 111.5)
 		(width 0.25)
 		(layer "B.Cu")
@@
 	)
 	(segment
-		(start 224.5 109.52)
-		(end 226.48 111.5)
+		(start 217.9 110.3)
+		(end 217.9 91.3)
 		(width 0.25)
 		(layer "B.Cu")
@@
 	)
 	(segment
+		(start 226.48 111.5)
+		(end 235.7 111.5)
+		(width 0.25)
+		(layer "B.Cu")
+		(net 17)
+	)
+	(segment
 		(start 223.5 109.52)
 		(end 224.5 109.52)
@@
 	)
 	(segment
+		(start 235.7 111.5)
+		(end 236.9 110.3)
+		(width 0.25)
+		(layer "B.Cu")
+		(net 17)
+	)
+	(segment
 		(start 256 110.2)
 		(end 256 97.96)
@@
 	)
 	(segment
-		(start 231.6554 40.9325)
-		(end 231.6154 40.8925)
-		(width 0.254)
+		(start 239.5 72.3)
+		(end 243.98 72.3)
+		(width 0.25)
 		(layer "B.Cu")
 		(net 18)
@@
 	)
 	(segment
-		(start 243.98 72.3)
-		(end 244.09 72.41)
-		(width 0.25)
-		(layer "B.Cu")
-		(net 18)
-	)
-	(segment
 		(start 233 65)
 		(end 217.71602 49.71602)
@@
 	)
 	(segment
-		(start 239.5 72.3)
-		(end 239.7 72.3)
-		(width 0.25)
-		(layer "B.Cu")
-		(net 18)
-	)
-	(segment
 		(start 61.4911 47.75)
 		(end 64.4625 47.75)
@@
 	)
 	(segment
-		(start 239.5 72.3)
-		(end 243.98 72.3)
-		(width 0.25)
-		(layer "B.Cu")
-		(net 18)
-	)
-	(segment
 		(start 255.2 54)
 		(end 255.9 53.3)
@@
 	)
 	(segment
-		(start 244.09 72.41)
-		(end 247 75.32)
-		(width 0.25)
-		(layer "B.Cu")
-		(net 18)
-	)
-	(segment
 		(start 236.9 72.3)
 		(end 233.8 72.3)
@@
 	)
 	(segment
+		(start 243.98 72.3)
+		(end 247 75.32)
+		(width 0.25)
+		(layer "B.Cu")
+		(net 18)
+	)
+	(segment
 		(start 217.71602 49.71602)
 		(end 217.71602 48.20352)
@@
 	)
 	(segment
-		(start 221 47.75)
-		(end 224.062402 47.75)
-		(width 0.254)
-		(locked yes)
-		(layer "B.Cu")
-		(net 21)
-	)
-	(segment
 		(start 34.5422 28.4211)
 		(end 34.085 27.9639)
@@
 	)
 	(segment
-		(start 72.63 93)
-		(end 72.59 92.96)
-		(width 0.254)
-		(layer "F.Cu")
-		(net 45)
-	)
-	(segment
 		(start 116.9875 48.0125)
 		(end 113.068479 51.931521)
@@
 	)
 	(segment
-		(start 149 55.638932)
-		(end 149 64.961374)
-		(width 0.254)
-		(layer "F.Cu")
-		(net 49)
-	)
-	(segment
 		(start 150.599511 47.562989)
 		(end 150.4125 47.75)
@@
 	)
 	(segment
-		(start 149 50.5)
-		(end 149 55.638932)
-		(width 0.254)
-		(layer "F.Cu")
-		(net 49)
-	)
-	(segment
 		(start 150.599511 41.739511)
 		(end 150.599511 47.562989)
@@
 	)
 	(segment
-		(start 148.902414 50.402414)
-		(end 149 50.5)
-		(width 0.254)
-		(layer "F.Cu")
-		(net 49)
-	)
-	(segment
-		(start 149 64.5)
-		(end 149 64.962053)
+		(start 150.4125 47.75)
+		(end 150.4125 48.892328)
 		(width 0.254)
+		(locked yes)
 		(layer "F.Cu")
 		(net 49)
 	)
 	(segment
-		(start 150.4125 47.75)
-		(end 150.4125 48.892328)
+		(start 149 50.304828)
+		(end 149 64.961374)
 		(width 0.254)
-		(locked yes)
 		(layer "F.Cu")
 		(net 49)
@@
 	(segment
 		(start 150.4125 48.892328)
-		(end 148.902414 50.402414)
+		(end 149 50.304828)
 		(width 0.254)
 		(layer "F.Cu")
@@
 	)
 	(segment
-		(start 194.853479 95.99257)
-		(end 194.853479 96.008043)
-		(width 0.254)
-		(locked yes)
-		(layer "F.Cu")
-		(net 55)
-	)
-	(segment
 		(start 189.5 59)
 		(end 189.5 106.85)
@@
 	)
 	(segment
-		(start 128.721957 46.124457)
-		(end 128.721957 75.173479)
+		(start 126.586521 77.308915)
+		(end 126 77.895436)
 		(width 0.254)
 		(layer "F.Cu")
@@
 	)
 	(segment
-		(start 126 99.15)
-		(end 115.9 109.25)
+		(start 128.721957 46.124457)
+		(end 128.721957 75.173479)
 		(width 0.254)
 		(layer "F.Cu")
@@
 	)
 	(segment
-		(start 126 77.895436)
-		(end 126 99.15)
+		(start 126 99.15)
+		(end 115.9 109.25)
 		(width 0.254)
 		(layer "F.Cu")
@@
 	)
 	(segment
-		(start 126.586521 77.308915)
-		(end 126 77.895436)
+		(start 126 77.895436)
+		(end 126 99.15)
 		(width 0.254)
 		(layer "F.Cu")
